File: controller/controller.kicad_pcb (KiCad board)
At the start: 2 copper layers, 69.6 x 37.3 mm, 65 parts, among them J1 Conn_01x25_Membrane, J2 Conn_01x04, J3 Conn_Solenoid_Driver, J4 Conn_01x01, J6 Conn_01x06, Q1 Q_PMOS_GSD AO3401A, Q2 Q_NMOS_GSD 2N7002, Q3 Q_NMOS_GSD 2N7002, SW1 SW_Push, U1 AMS1117-3.3, U2 STM32F446RETx, U3 TPS2553DBVR, U4 USBLC6-2SC6, U5 24LC64, Y1 16MHz

Commit message: fix
Parts:
- removed J2: Conn_01x04, Connector_JST:JST_PH_S4B-PH-K_1x04_P2.00mm_Horizontal
- removed R1: 390, Resistor_SMD:R_0805_2012Metric_Pad1.15x1.40mm_HandSolder
- added J5: Conn_01x04_MountingPin, Connector_JST:JST_SH_SM04B-SRSS-TB_1x04-1MP_P1.00mm_Horizontal, F.Cu at (122.9, 137.5)
- U2: value STM32F446RETx -> STM32F401RETx
- U4: footprint Package_TO_SOT_SMD:SOT-666 -> Package_TO_SOT_SMD:SOT-23-6
- Y1: value 16MHz -> 8MHz
- moved U4 2.49 mm to (121.2, 144.0)
Connections:
- net /VCAP_1 renamed Net-(U2-VCAP1)
- C9 pad 1: /OSCO_RES -> /OSCO
- R4 pad 2: LEDDRV2_USART3RX_BL -> unconnected-(R4-Pad2)
- SW1 pad 2: Net-(SW1-Pad2) -> unconnected-(SW1-Pad2)
- SW1 pad 3: Net-(SW1-Pad3) -> unconnected-(SW1-Pad3)
- U2 pad 12: GND -> unconnected-(U2-VSSA)
- U2 pad 18: GND -> unconnected-(U2-VSS)_1
- U2 pad 3: Net-(U2-Pad3) -> unconnected-(U2-PC14)
- U2 pad 31: GND -> unconnected-(U2-VSS)_2
- U2 pad 4: Net-(U2-Pad4) -> unconnected-(U2-PC15)
- U2 pad 46: Net-(U2-Pad46) -> unconnected-(U2-PA13)
- U2 pad 47: GND -> unconnected-(U2-VSS)_3
- U2 pad 59: Net-(U2-Pad59) -> unconnected-(U2-PB7)
- U2 pad 60: /BOOT0 -> unconnected-(U2-BOOT0)
- U2 pad 61: Net-(U2-Pad61) -> unconnected-(U2-PB8)
- U2 pad 63: GND -> unconnected-(U2-VSS)
- U2 pad 7: /NRST -> unconnected-(U2-NRST)
- Y1 pad 3: /OSCO_RES -> /OSCO
Routing:
- net unconnected-(J5-MountPin): track 0.00 -> 7.60 mm, vias 0 -> 2
- net /OSCO: track 2.86 -> 9.36 mm
- net /OSCO_RES: track 5.27 -> 0.00 mm
- net unconnected-(U2-VSS)_3: track 0.00 -> 2.28 mm, vias 0 -> 1
- net GND: track 27.1 -> 25.5 mm, vias 236 -> 217
- net VBUS: track 65.2 -> 63.8 mm
- net USB_DP: track 10.3 -> 9.29 mm
- net USB_DP_ESD: track 3.35 -> 3.93 mm
Other:
- net class Default removed
- board text added: "4.3mm holes"
- board text added: "Replacement controller for Model M keyboards djvs unified daughterboard/stm32f401retx modifications"
- board text removed: "3.2mm holes"
- board text removed: "Replacement controller for Model M keyboards"
